Commit message: Fixed the orientation of the servos in the leg. One was flipped 180 degrees.

File: solidworks/urdf_output/WalkBot/urdf/WalkBot.urdf (robot description, URDF)
Before this commit: robot WalkBot, 7 links, 6 joints
Links:
- link Body: mass 0.520746828527768 -> 0.52075
- link Servo1_Right: mass 0.0230007365895397 -> 0
- link Servo2_Left: mass 0.0226043083522871 -> 0.022604308352287
Joints:
- joint ankle_R: origin xyz=0 -0.047416 0 rpy=0 0 0 -> xyz=0 -0.0474161341528267 0 rpy=0 0 0
- joint hip_R: origin xyz=-0.05 -0.048627 0 rpy=0 0 0 -> xyz=-0.05 -0.0486271117592205 0 rpy=0 0 0
- joint knee_R: origin xyz=0 -0.047416 0 rpy=0 0 0 -> xyz=0 -0.0474161341528266 0 rpy=0 0 0

Commit message: The rotation axis for the leg joints were still wrong, needed to be changed in the URDF exporter. This version should be correct

File: solidworks/urdf_output/WalkBot/urdf/WalkBot.urdf (robot description, URDF)
Before this commit: robot WalkBot, 7 links, 6 joints
Links:
- link Servo1_Left: mass 0.0230007365895397 -> 0.023001
- link Servo1_Right: mass 0 -> 0.023001
- link Servo2_Left: mass 0.022604308352287 -> 0.022604
- link Servo2_Right: mass 0.0226043083522871 -> 0.022604
- link Servo3_Left: mass 0.0161002375604621 -> 0.0161
- link Servo3_Right: mass 0.0161002375604621 -> 0.0161
Joints:
- joint ankle_R: origin xyz=0 -0.0474161341528267 0 rpy=0 0 0 -> xyz=0 -0.047416 0 rpy=0 0 0
- joint hip_R: origin xyz=-0.05 -0.0486271117592205 0 rpy=0 0 0 -> xyz=-0.05 -0.048627 0 rpy=0 0 0
- joint knee_L: axis -1 0 0 -> 1 0 0
- joint knee_R: axis -1 0 0 -> 1 0 0; origin xyz=0 -0.0474161341528266 0 rpy=0 0 0 -> xyz=0 -0.047416 0 rpy=0 0 0

Commit message: The coordinate systems were oriented incorrectly. They've been updated so Z is up, X is forward. Additionally the Body now has an arrow feature to indicate the front of the bot

File: solidworks/urdf_output/WalkBot/urdf/WalkBot.urdf (robot description, URDF)
Before this commit: robot WalkBot, 7 links, 6 joints
Links:
- link Body: mass 0.52075 -> 0.51911
Joints:
- joint ankle_L: axis 1 0 0 -> 0 1 0; origin xyz=0 -0.047416 0 rpy=0 0 0 -> xyz=0 0 -0.047416 rpy=0 0 0
- joint ankle_R: axis 1 0 0 -> 0 1 0; origin xyz=0 -0.047416 0 rpy=0 0 0 -> xyz=0 0 -0.047416 rpy=0 0 0
- joint hip_L: axis 0 0 1 -> 1 0 0; origin xyz=0.05 -0.048627 0 rpy=0 0 0 -> xyz=0 0.05 -0.048627 rpy=0 0 0
- joint hip_R: axis 0 0 1 -> 1 0 0; origin xyz=-0.05 -0.048627 0 rpy=0 0 0 -> xyz=0 -0.05 -0.048627 rpy=0 0 0
- joint knee_L: axis 1 0 0 -> 0 1 0; origin xyz=0 -0.047416 0 rpy=0 0 0 -> xyz=0 0 -0.047416 rpy=0 0 0
- joint knee_R: axis 1 0 0 -> 0 1 0; origin xyz=0 -0.047416 0 rpy=0 0 0 -> xyz=0 0 -0.047416 rpy=0 0 0
