Commit message: Update from the Linux end. Just some cleaning up.

File: assets/urdf/WalkBot/urdf/WalkBot.urdf (robot description, URDF)
Before this commit: robot WalkBot, 7 links, 6 joints
Links:
- removed link body
- removed link servo1l
- removed link servo1r
- removed link servo2l
- removed link servo2r
- removed link servo3l
- removed link servo3r
- added link Body, mass 0.52075; collision mesh filename=../meshes/Body.STL; visual mesh filename=../meshes/Body.STL
- added link Servo1_Left, mass 0.0230007365895397; collision mesh filename=../meshes/Servo1_Left.STL; visual mesh filename=../meshes/Servo1_Left.STL
- added link Servo1_Right, mass 0; collision mesh filename=../meshes/Servo1_Right.STL; visual mesh filename=../meshes/Servo1_Right.STL
- added link Servo2_Left, mass 0.022604308352287; collision mesh filename=../meshes/Servo2_Left.STL; visual mesh filename=../meshes/Servo2_Left.STL
- added link Servo2_Right, mass 0.0226043083522871; collision mesh filename=../meshes/Servo2_Right.STL; visual mesh filename=../meshes/Servo2_Right.STL
- added link Servo3_Left, mass 0.0161002375604621; collision mesh filename=../meshes/Servo3_Left.STL; visual mesh filename=../meshes/Servo3_Left.STL
- added link Servo3_Right, mass 0.0161002375604621; collision mesh filename=../meshes/Servo3_Right.STL; visual mesh filename=../meshes/Servo3_Right.STL
Joints:
- removed joint anklel
- removed joint ankler
- removed joint hipl
- removed joint hipr
- removed joint kneel
- removed joint kneer
- added joint ankle_L: type revolute, parent Servo2_Left, child Servo3_Left, origin xyz=0 -0.047416 0 rpy=0 0 0, axis 1 0 0, limit lower=-1.5708 upper=1.5708 effort=0.52 velocity=10.89
- added joint ankle_R: type revolute, parent Servo2_Right, child Servo3_Right, origin xyz=0 -0.0474161341528267 0 rpy=0 0 0, axis 1 0 0, limit lower=-1.5708 upper=1.5708 effort=0.52 velocity=10.89
- added joint hip_L: type revolute, parent Body, child Servo1_Left, origin xyz=0.05 -0.048627 0 rpy=0 0 0, axis 0 0 1, limit lower=-1.5708 upper=1.5708 effort=0.52 velocity=10.89
- added joint hip_R: type revolute, parent Body, child Servo1_Right, origin xyz=-0.05 -0.0486271117592205 0 rpy=0 0 0, axis 0 0 1, limit lower=-1.5708 upper=1.5708 effort=0.52 velocity=10.89
- added joint knee_L: type revolute, parent Servo1_Left, child Servo2_Left, origin xyz=0 -0.047416 0 rpy=0 0 0, axis -1 0 0, limit lower=-1.5708 upper=1.5708 effort=0.52 velocity=10.89
- added joint knee_R: type revolute, parent Servo1_Right, child Servo2_Right, origin xyz=0 -0.0474161341528266 0 rpy=0 0 0, axis -1 0 0, limit lower=-1.5708 upper=1.5708 effort=0.52 velocity=10.89

File: assets/urdf/WalkBot_3DOF_330/urdf/WalkBot_3DOF.urdf (robot description, URDF)
Before this commit: robot Robot, 7 links, 6 joints
Links:
- removed link body
- removed link servo1l
- removed link servo1r
- removed link servo2l
- removed link servo2r
- removed link servo3l
- removed link servo3r
- added link Ankle_L, mass 0.0318831730757301; collision mesh filename=../meshes/Ankle_L.STL; visual mesh filename=../meshes/Ankle_L.STL
- added link Ankle_R, mass 0.0318831730757301; collision mesh filename=../meshes/Ankle_R.STL; visual mesh filename=../meshes/Ankle_R.STL
- added link Body, mass 0.520746828527768; collision mesh filename=../meshes/Body.STL; visual mesh filename=../meshes/Body.STL
- added link Hip_L, mass 0.0230007365895397; collision mesh filename=../meshes/Hip_L.STL; visual mesh filename=../meshes/Hip_L.STL
- added link Hip_R, mass 0.0230007365895397; collision mesh filename=../meshes/Hip_R.STL; visual mesh filename=../meshes/Hip_R.STL
- added link Knee_L, mass 0.022604308352287; collision mesh filename=../meshes/Knee_L.STL; visual mesh filename=../meshes/Knee_L.STL
- added link Knee_R, mass 0.022604308352287; collision mesh filename=../meshes/Knee_R.STL; visual mesh filename=../meshes/Knee_R.STL
Joints:
- removed joint anklel
- removed joint ankler
- removed joint hipl
- removed joint hipr
- removed joint kneel
- removed joint kneer
- added joint Ankle_L: type revolute, parent Knee_L, child Ankle_L, origin xyz=0 -0.0473161341528267 0 rpy=0 0 0, axis 1 0 0, limit lower=-1.57 upper=1.57 effort=0.52 velocity=10.89
- added joint Ankle_R: type revolute, parent Knee_R, child Ankle_R, origin xyz=0 -0.0473161341528267 0 rpy=0 0 0, axis -1 0 0, limit lower=-1.57 upper=1.57 effort=0.52 velocity=10.89
- added joint Hip_L: type revolute, parent Body, child Hip_L, origin xyz=0.0500000000000003 -0.0581271117592202 0.000499999999998217 rpy=0 0 0, axis 0 0 1, limit lower=-1.57 upper=1.57 effort=0.52 velocity=10.89
- added joint Hip_R: type revolute, parent Body, child Hip_R, origin xyz=-0.05 -0.058127 0.0005 rpy=0 0 0, axis 0 0 1, limit lower=-1.57 upper=1.57 effort=0.52 velocity=10.89
- added joint Knee_L: type revolute, parent Hip_L, child Knee_L, origin xyz=0.000500000000000216 -0.0473161341528267 -0.000500000000000007 rpy=0 0 0, axis 1 0 0, limit lower=-1.57 upper=1.57 effort=0.52 velocity=10.89
- added joint Knee_R: type revolute, parent Hip_R, child Knee_R, origin xyz=0.0005 -0.047316 -0.0005 rpy=0 0 0, axis -1 0 0, limit lower=-1.57 upper=1.57 effort=0.52 velocity=10.89

Commit message: Training looks like it is working properly for position control. Still need to take a look at why Torque control was having poor results

File: assets/urdf/WalkBot/urdf/WalkBot.urdf (robot description, URDF)
Before this commit: robot WalkBot, 7 links, 6 joints
Links:
- link Body: mass 0.52075 -> 0.51911
- link Servo1_Left: mass 0.0230007365895397 -> 0.023001
- link Servo1_Right: mass 0 -> 0.023001
- link Servo2_Left: mass 0.022604308352287 -> 0.022604
- link Servo2_Right: mass 0.0226043083522871 -> 0.022604
- link Servo3_Left: mass 0.0161002375604621 -> 0.0161
- link Servo3_Right: mass 0.0161002375604621 -> 0.0161
Joints:
- joint ankle_L: axis 1 0 0 -> 0 1 0; origin xyz=0 -0.047416 0 rpy=0 0 0 -> xyz=0 0 -0.047416 rpy=0 0 0
- joint ankle_R: axis 1 0 0 -> 0 1 0; origin xyz=0 -0.0474161341528267 0 rpy=0 0 0 -> xyz=0 0 -0.047416 rpy=0 0 0
- joint hip_L: axis 0 0 1 -> 1 0 0; origin xyz=0.05 -0.048627 0 rpy=0 0 0 -> xyz=0 0.05 -0.048627 rpy=0 0 0
- joint hip_R: axis 0 0 1 -> 1 0 0; origin xyz=-0.05 -0.0486271117592205 0 rpy=0 0 0 -> xyz=0 -0.05 -0.048627 rpy=0 0 0
- joint knee_L: axis -1 0 0 -> 0 1 0; origin xyz=0 -0.047416 0 rpy=0 0 0 -> xyz=0 0 -0.047416 rpy=0 0 0
- joint knee_R: axis -1 0 0 -> 0 1 0; origin xyz=0 -0.0474161341528266 0 rpy=0 0 0 -> xyz=0 0 -0.047416 rpy=0 0 0
