Commit message: Added the work from the WalkBot_IKRL project. This was getting the foot to touch a goal point. I also started adding in sound code to try out on the jetson. I think this might be a good foundation to start running the learned policy on hardware. The model looks like it is being loaded and I can feed in fake observations. Next step will be running on the Jetson, Timing the loop, get getting REAL observationsgit status! :)

File: assets/urdf/WalkBot_IKRL/urdf/WalkBot.urdf (robot description, URDF)
Before this commit: robot WalkBot, 7 links, 6 joints
Links:
- removed link Servo1_Left
- removed link Servo2_Left
- removed link Servo3_Left
Joints:
- removed joint ankle_L
- removed joint hip_L
- removed joint knee_L
