Commit message: Updated walkbot 4 leg coordinate system. Z Up...

File: solidworks/urdf_output/WalkBot4Leg/urdf/WalkBot4Leg.urdf (robot description, URDF)
Before this commit: robot WalkBot4Leg.SLDASM, 13 links, 12 joints
Links:
- link BL1_Servo: geometry collision mesh filename=package://WalkBot4Leg/meshes/BL1_Servo.STL; visual mesh filename=package://WalkBot4Leg/meshes/BL1_Servo.STL
- link BL2_Servo: geometry collision mesh filename=package://WalkBot4Leg/meshes/BL2_Servo.STL; visual mesh filename=package://WalkBot4Leg/meshes/BL2_Servo.STL
- link BL3_Servo: geometry collision mesh filename=package://WalkBot4Leg/meshes/BL3_Servo.STL; visual mesh filename=package://WalkBot4Leg/meshes/BL3_Servo.STL
- link BR1_Servo: geometry collision mesh filename=package://WalkBot4Leg/meshes/BR1_Servo.STL; visual mesh filename=package://WalkBot4Leg/meshes/BR1_Servo.STL
- link BR2_Servo: geometry collision mesh filename=package://WalkBot4Leg/meshes/BR2_Servo.STL; visual mesh filename=package://WalkBot4Leg/meshes/BR2_Servo.STL
- link BR3_Servo: geometry collision mesh filename=package://WalkBot4Leg/meshes/BR3_Servo.STL; visual mesh filename=package://WalkBot4Leg/meshes/BR3_Servo.STL
- link Body: geometry collision mesh filename=package://WalkBot4Leg/meshes/Body.STL; visual mesh filename=package://WalkBot4Leg/meshes/Body.STL
- link FL1_Servo: geometry collision mesh filename=package://WalkBot4Leg/meshes/FL1_Servo.STL; visual mesh filename=package://WalkBot4Leg/meshes/FL1_Servo.STL
- link FL2_Servo: geometry collision mesh filename=package://WalkBot4Leg/meshes/FL2_Servo.STL; visual mesh filename=package://WalkBot4Leg/meshes/FL2_Servo.STL
- link FL3_Servo: geometry collision mesh filename=package://WalkBot4Leg/meshes/FL3_Servo.STL; visual mesh filename=package://WalkBot4Leg/meshes/FL3_Servo.STL
- link FR1_Servo: geometry collision mesh filename=package://WalkBot4Leg/meshes/FR1_Servo.STL; visual mesh filename=package://WalkBot4Leg/meshes/FR1_Servo.STL
- link FR2_Servo: geometry collision mesh filename=package://WalkBot4Leg/meshes/FR2_Servo.STL; visual mesh filename=package://WalkBot4Leg/meshes/FR2_Servo.STL
- link FR3_Servo: geometry collision mesh filename=package://WalkBot4Leg/meshes/FR3_Servo.STL; visual mesh filename=package://WalkBot4Leg/meshes/FR3_Servo.STL
Joints:
- joint BL1: axis 0 0 1 -> 1 0 0; origin xyz=0.05 -0.0488561341528267 -0.071 rpy=0 0 0 -> xyz=-0.071 0.05 -0.0488561341528267 rpy=0 0 0
- joint BL2: axis -1 0 0 -> 0 -1 0; origin xyz=0 -0.0474161341528266 0 rpy=0 0 0 -> xyz=0 0 -0.0474161341528266 rpy=0 0 0
- joint BL3: axis -1 0 0 -> 0 -1 0; origin xyz=0 -0.0474161341528267 0 rpy=0 0 0 -> xyz=0 0 -0.0474161341528267 rpy=0 0 0
- joint BR1: axis 0 0 1 -> 1 0 0; origin xyz=-0.05 -0.048856 -0.071 rpy=0 0 0 -> xyz=-0.071 -0.05 -0.048856 rpy=0 0 0
- joint BR2: axis -1 0 0 -> 0 -1 0; origin xyz=0 -0.0474161341528266 0 rpy=0 0 0 -> xyz=0 0 -0.0474161341528266 rpy=0 0 0
- joint BR3: axis -1 0 0 -> 0 -1 0; origin xyz=0 -0.0474161341528267 0 rpy=0 0 0 -> xyz=0 0 -0.0474161341528267 rpy=0 0 0
- joint FL1: axis 0 0 1 -> 1 0 0; origin xyz=0.05 -0.048856 0.071 rpy=0 0 0 -> xyz=0.071 0.05 -0.048856 rpy=0 0 0
- joint FL2: axis -1 0 0 -> 0 -1 0; origin xyz=0 -0.0474161341528266 0 rpy=0 0 0 -> xyz=0 0 -0.0474161341528266 rpy=0 0 0
- joint FL3: axis -1 0 0 -> 0 -1 0; origin xyz=0 -0.0474161341528267 0 rpy=0 0 0 -> xyz=0 0 -0.0474161341528267 rpy=0 0 0
- joint FR1: axis 0 0 1 -> 1 0 0; origin xyz=-0.05 -0.048856 0.071 rpy=0 0 0 -> xyz=0.071 -0.05 -0.048856 rpy=0 0 0
- joint FR2: axis -1 0 0 -> 0 -1 0; origin xyz=0 -0.047416 0 rpy=0 0 0 -> xyz=0 0 -0.047416 rpy=0 0 0
- joint FR3: axis -1 0 0 -> 0 -1 0; origin xyz=0 -0.047416 0 rpy=0 0 0 -> xyz=0 0 -0.0474161341528267 rpy=0 0 0
